File: schematics/fornoSmart/pwr.kicad_sch (KiCad schematic)
At the start: 12 parts, among them J3 LineIn, J3-A rele, J7 Controlador, K1 Fujitsu_FTR-LYAA005x, K2 Fujitsu_FTR-LYAA005x, K3 Fujitsu_FTR-LYAA005x, Q2 TIP120

Commit message: 2025-12 update
Parts:
- removed K3: Fujitsu_FTR-LYAA005x, Relay_THT:Relay_SPST-NO_Fujitsu_FTR-LYAA005x_FormA_Vertical, symbol Relay:Fujitsu_FTR-LYAA005x
- added U1: HHG1D-1, Relay_THT:Relay_NCR_HHG1D-1, symbol Relay_SolidState:HHG1D-1
- J3-A: value rele -> ControladorIN
- J7: value Controlador -> ControladorOut
Connections:
- net Linha: now also U1.1; no longer K1.14
- net at K1.13: no longer R2.1
- net heater_line: now reaches R3.1
- net heater_line: now also R2.1, U1.2
- net Neutro renamed heater_netro
Other:
- moved on the sheet: D1, J3, J3-A, J7, K1, K2, PS1, Q2, R1, R2, R3
