File: fornoSmartEsp32/schematics/fornoSmart/fs.kicad_sch (KiCad schematic)
At the start: 17 parts, among them J1 display, J10 LineIn, J11 ControladorOUT, J12 ReleTempControll, J13 heaters, J14 ReleTempControll, J4 speaker, J5 led, J6 VIN-5V, K3 Fujitsu_FTR-LYAA005x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

Commit message: Updating...
Parts:
- removed J10: LineIn, symbol Connector_Generic:Conn_01x02
- removed J11: ControladorOUT, symbol Connector_Generic:Conn_01x02
- removed J12: ReleTempControll, symbol Connector_Generic:Conn_01x02
- removed J13: heaters, symbol Connector_Generic:Conn_01x02
- removed K3: Fujitsu_FTR-LYAA005x, Relay_THT:Relay_SPST-NO_Fujitsu_FTR-LYAA005x_FormA_Vertical, symbol Relay:Fujitsu_FTR-LYAA005x
- removed PS2: 127_220_x_05V, Converter_DCDC:Converter_DCDC_XP_POWER-ITXxxxxSA_THT, symbol Converter_DCDC:ITX1209SA
- removed R4: assar, symbol Device:Heater
- removed R5: Dourador, symbol Device:Heater
- removed U2: HHG1D-1, Relay_THT:Relay_NCR_HHG1D-1, symbol Relay_SolidState:HHG1D-1
Other:
- note removed: "Montado no interior tampa traseira."
- note removed: "Painel Frontal"
