File: fornoSmartEsp32/schematics/fornoSmart/pwr.kicad_sch (KiCad schematic)
At the start: 14 parts, among them J3 LineIn, J3-A ControladorIN, J7 ControladorIN, J8 heaters, J9 ControladorOUT, K1 Fujitsu_FTR-LYAA005x, K2 Fujitsu_FTR-LYAA005x, Q2 TIP120, U1 HHG1D-1

Commit message: Updating...
Parts:
- removed J3: LineIn, symbol Connector_Generic:Conn_01x02
- removed J7: ControladorIN, symbol Connector_Generic:Conn_01x02
- removed J8: heaters, symbol Connector_Generic:Conn_01x02
- removed J9: ControladorOUT, symbol Connector_Generic:Conn_01x02
- removed K1: Fujitsu_FTR-LYAA005x, Relay_THT:Relay_SPST-NO_Fujitsu_FTR-LYAA005x_FormA_Vertical, symbol Relay:Fujitsu_FTR-LYAA005x
- added SW3: switch_dourador, symbol Switch:SW_SPDT_XKB_DMx-xxxx-1
- added TH1: PT100, symbol Sensor_Temperature:PT100
- PSU1: renamed from PS1; value 127_220_x_05V -> POWER_SUPPLAY_127-5V
- U1: value HHG1D-1 -> SSD
Connections:
- net heater_line is gone; now on net LINE: U1.1
- net +5V: now also J3-A.1 (Pin_1)
- net GND: now also J3-A.3 (Pin_3); no longer U1.4
- net Linha renamed LINE
- net Neutro renamed NEUTRO 
- net NEUTRO : now also R2.1, SW3.1 (A)
- net heater_netro: no longer names the net of R2.2, R3.2
- net heater_netro: now also U1.2
- new net: R3.1, SW3.2 (B)
Other:
- note added: "1"
- note added: "10"
- note added: "2"
- note added: "3"
- note added: "4"
- note added: "9"
- moved on the sheet: D1, J3-A, K2, PSU1, Q2, R1, R2, R3, U1
